Commit message: sim

File: src/motor/description/motor_design.xacro (robot description, xacro)
@@ -1,4 +1,4 @@
 <?xml version="1.0"?>
-<robot xmlns:xacro="http://www.ros.org/wiki/xacro" name="robosi">
+<robot xmlns:xacro="http://www.ros.org/wiki/xacro">
     <!-- Robot size -->
     <!-- Length = 300mm-->
@@ -8,4 +8,5 @@
     <link name="base_link">
     </link>
+    <!-- CHASSIS LINK -->
     <joint name="chassis_joint" type="fixed">
         <parent link="base_link"/>
@@ -31,4 +32,17 @@
         </xacro:inertial_box>
     </link>
+    <!-- <gazebo reference="chassis_link">
+        <material>Gazebo/Grey</material>
+    </gazebo> -->
+    <gazebo reference="chassis_link">
+        <visual>
+            <material>
+                <ambient>0.8509 0.8431 0.7921 1.0</ambient>
+                <diffuse>0.8509 0.8431 0.7921 1.0</diffuse>
+                <specular>0.8509 0.8431 0.7921 1.0 1.0</specular>
+                <!-- <emissive>15/255 6/255 179/255 1</emissive> -->
+            </material>
+        </visual>
+    </gazebo>
     <!-- LEFT WHEEL -->
     <joint name="left_wheel_joint" type="continuous">
@@ -56,4 +70,13 @@
         </xacro:inertial_cylinder>
     </link>
+    <gazebo reference="left_wheel_link">
+        <visual>
+            <material>
+                <ambient>0.2353 0.5529 0.5764 1.0</ambient>
+                <diffuse>0.2353 0.5529 0.5764 1.0</diffuse>
+                <specular>0.2353 0.5529 0.5764 1.0 1.0</specular>
+            </material>
+        </visual>
+    </gazebo>
     <!-- RIGHT WHEEL -->
     <joint name="right_wheel_joint" type="continuous">
@@ -81,4 +104,13 @@
         </xacro:inertial_cylinder>
     </link>
+    <gazebo reference="right_wheel_link">
+        <visual>
+            <material>
+                <ambient>0.2353 0.5529 0.5764 1.0</ambient>
+                <diffuse>0.2353 0.5529 0.5764 1.0</diffuse>
+                <specular>0.2353 0.5529 0.5764 1.0 1.0</specular>
+            </material>
+        </visual>
+    </gazebo>
     <!-- CASTER WHEEL -->
     <joint name="caster_wheel_joint" type="fixed">
@@ -105,3 +137,14 @@
         </xacro:inertial_sphere>
     </link>
+    <gazebo reference="caster_wheel_link">
+        <visual>
+            <material>
+                <ambient>0.2313 0.2078 0.2078 1.0</ambient>
+                <diffuse>0.2313 0.2078 0.2078 1.0</diffuse>
+                <specular>0.2313 0.2078 0.2078 1.0 1.0</specular>
+            </material>
+        </visual>
+        <mu1 value="0.001"/>
+        <mu2 value="0.001"/>
+    </gazebo>
 </robot>

File: src/motor/description/motor_functions.xacro (robot description, xacro)
@@ -3,17 +3,17 @@
     <!-- Colors -->
     <material name="WhiteGrey">
-        <color rgba="${217/255} ${215/255} ${202/255} 1.0" />
+        <color rgba="${217/255} ${215/255} ${202/255} 1.0" /> **0.8509 0.8431 0.7921 1.0**
     </material>
     <material name="LightBlueGreen">
-        <color rgba="${60/255} ${141/255} ${147/255} 1.0" />
+        <color rgba="${60/255} ${141/255} ${147/255} 1.0" />**0.2353 0.5529 0.5764 1.0**
     </material>
     <material name="DarkBlueGreen">
-        <color rgba="${31/255} ${69/255} ${77/255} 1.0" />
+        <color rgba="${31/255} ${69/255} ${77/255} 1.0" />**0.1215 0.2705 0.3019 1.0**
     </material>
     <material name="Brown">
-        <color rgba="${115/255} ${96/255} ${79/255} 1.0" />
+        <color rgba="${115/255} ${96/255} ${79/255} 1.0" />**0.4509 0.3764 0.3098 1.0**
     </material>
     <material name="BrownBlack">
-        <color rgba="${59/255} ${53/255} ${53/255} 1.0" />
+        <color rgba="${59/255} ${53/255} ${53/255} 1.0" />**0.2313 0.2078 0.2078 1.0**
     </material>
     <!-- Define equations that calculate the inertias-->

Commit message: updates

File: src/motor/description/motor_design.xacro (robot description, xacro)
@@ -123,5 +123,5 @@
             <origin xyz="0.0 0.0 0.0" rpy="0.0 0.0 0.0"/>
             <geometry>
-                <sphere radius="0.04"/>
+                <sphere radius="0.05"/>
             </geometry>
             <material name="BrownBlack"/>
